File: WemosD1_Iobroker_Adapter/WemosD1_Iobroker_Adapter.kicad_pcb (KiCad board)
At the start: 2 copper layers, 25.9 x 39.6 mm, 26 parts, among them J1 Conn_01x12_Female, U1 WeMos_D1_mini, U2 LM393, U3 LP2985-3.3, U4 6N136S

Commit message: initial commit
Parts:
- added C8: 470p, Capacitor_SMD:C_0402_1005Metric, F.Cu at (118.5, 55.5)
- added R11: 330, Resistor_SMD:R_0402_1005Metric, F.Cu at (114.0, 59.3)
- C5: footprint Capacitor_SMD:C_0402_1005Metric -> Capacitor_SMD:C_0603_1608Metric
- U2: footprint Package_SO:MSOP-8_3x3mm_P0.65mm -> Package_SO:SOIC-8_3.9x4.9mm_P1.27mm
- moved C5 20.8 mm to (106.2, 36.0)
- moved R8 5.86 mm to (121.2, 39.8)
- moved R5 1.75 mm to (111.7, 50.5)
- moved R6 1.30 mm to (115.2, 45.3)
- moved C6 1.22 mm to (110.0, 51.0)
- moved R4 1.22 mm to (110.0, 50.0)
- moved R7 1.20 mm to (113.0, 45.3)
- moved U2 1.01 mm to (115.2, 49.8)
- moved U4 1.00 mm to (114.2, 38.0)
- moved R9 0.90 mm to (106.9, 58.9)
- moved JP1 0.81 mm to (121.8, 50.9)
- moved D3 0.35 mm to (111.8, 59.6)
Connections:
- D3 pad 2: +VDC -> Net-(D3-Pad2)
- J1 pad 12: unconnected-(J1-Pad12) -> DS18B20_GND
- U3 pad 4: unconnected-(U3-Pad4) -> Net-(C8-Pad1)
Routing:
- net VBUS: track 10.7 -> 27.2 mm
- net Net-(U2-Pad1): track 0.00 -> 16.5 mm, vias 0 -> 2
- net +3V3: track 18.0 -> 34.1 mm, vias 0 -> 2
- net 3V3_WEMOS: track 26.0 -> 36.7 mm, vias 1 -> 0
- net DS18B20_GND: track 22.8 -> 15.5 mm, vias 0 -> 2
- net Net-(C6-Pad1): track 8.76 -> 11.7 mm
- net Net-(C8-Pad1): track 0.00 -> 2.81 mm
- net Net-(R8-Pad2): track 0.00 -> 2.27 mm
- net Net-(D1-Pad2): track 13.6 -> 11.9 mm
- net Net-(R5-Pad2): track 7.49 -> 8.94 mm
- net Net-(D3-Pad2): track 0.00 -> 1.37 mm
- net +VDC: track 23.5 -> 22.5 mm
- net VBUS+: track 10.4 -> 11.2 mm
- net GAS_SENSOR_INPUT: track 19.6 -> 19.0 mm
- net DS18B20_GPIO: track 5.64 -> 5.12 mm
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- added copper zone on B.Cu, net DS18B20_GND
- added copper zone on B.Cu, net GND
Other:
- board size 25.9 x 39.6 mm -> 26 x 39.5 mm
- board text added: "3V3"
- board text added: "5V"
- board text added: "DS"
- board text added: "GAS"
- board text added: "GND"
- board text added: "JLCJLCJLCJLC"
- board text added: "RX"
- board text added: "TX"
- board text added: "V+"
- board text added: "V-"
- board text added: "VBus/DS18B20/ SML/GAS/.V1 Oliver Horn horn.oliver@gmail.com"
