File: WemosD1_Iobroker_Adapter/WemosD1_Iobroker_Adapter.kicad_sch (KiCad schematic)
At the start: 26 parts, among them J1 Conn_01x12_Female, U1 WeMos_D1_mini, U2 LM393, U3 LP2985-3.3, U4 6N136S

Commit message: initial commit
Parts:
- added C8: 470p, Capacitor_SMD:C_0402_1005Metric, symbol Device:C
- added R11: 330, Resistor_SMD:R_0402_1005Metric, symbol Device:R
- C1, C2, C6, C7, D1, D2, D3, R1, R2, R3, R4, R5, R6, R7, R8, R9, U3, U4: now in the parts list
- C3, C4: LCSC Part # C60474 -> C307331; now in the parts list
- C5: footprint Capacitor_SMD:C_0402_1005Metric -> Capacitor_SMD:C_0603_1608Metric; LCSC Part # C1541 -> C1630; now in the parts list
- J1: LCSC Part # (none) -> C492434
- U1: now left out of the parts list
- U2: footprint Package_SO:MSOP-8_3x3mm_P0.65mm -> Package_SO:SOIC-8_3.9x4.9mm_P1.27mm; LCSC Part # C2688712 -> C7955; now in the parts list
Connections:
- net +VDC: now also R11.2; no longer D3.2 (K2)
- net GND: now also C8.2
- net GNDD: now also J1.12 (Pin_12)
- net at U3.4 (BP): now also C8.1
- net 5V_WEMOS renamed +5V
- new net: D3.2 (K2), R11.1
- no-connect marks 15 -> 13
Other:
- moved on the sheet: C1, C3, C4, C7, U3
